File: AnalogVideo.sch (KiCad schematic (older format))
At the start: 99 parts, among them Q101 2SA1462, Q102 DTA144EKA, Q103 2SC3545, Q201 2SA1462, Q202 DTA144EKA, Q203 2SC3545, Q301 2SA1462, Q302 DTA144EKA, Q303 2SC3545, Q401 2SC2412K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

Commit message: Switched to 8mm caps for video which should fit SMD bipolar ecaps
Parts:
- C103, C203, C303, C403: footprint Capacitors_SMD:CP_Elec_5x5.7 -> Capacitors_SMD:CP_Elec_8x5.4
Changed lines of the file:
@@
 F 0 "C103" V 5500 1200 50  0000 L CNN
 F 1 "47uF/16V/BP" V 5600 1200 50  0000 L CNN
-F 2 "Capacitors_SMD:CP_Elec_5x5.7" H 5700 1300 50  0001 C CNN
+F 2 "Capacitors_SMD:CP_Elec_8x5.4" H 5700 1300 50  0001 C CNN
 F 3 "" H 5700 1300 50  0001 C CNN
 	1    5700 1300
@@
 F 0 "C203" V 5500 3150 50  0000 L CNN
 F 1 "47uF/16V/BP" V 5600 3150 50  0000 L CNN
-F 2 "Capacitors_SMD:CP_Elec_5x5.7" H 5700 3250 50  0001 C CNN
+F 2 "Capacitors_SMD:CP_Elec_8x5.4" H 5700 3250 50  0001 C CNN
 F 3 "" H 5700 3250 50  0001 C CNN
 	1    5700 3250
@@
 F 0 "C303" V 5450 5150 50  0000 L CNN
 F 1 "47uF/16V/BP" V 5550 5150 50  0000 L CNN
-F 2 "Capacitors_SMD:CP_Elec_5x5.7" H 5700 5200 50  0001 C CNN
+F 2 "Capacitors_SMD:CP_Elec_8x5.4" H 5700 5200 50  0001 C CNN
 F 3 "" H 5700 5200 50  0001 C CNN
 	1    5700 5200
@@
 Connection ~ 4700 2350
 $Comp
-L VDDA #PWR048
+L VDDA #PWR049
 U 1 1 5E15C363
 P 4550 700
-F 0 "#PWR048" H 4550 550 50  0001 C CNN
+F 0 "#PWR049" H 4550 550 50  0001 C CNN
 F 1 "VDDA" V 4550 900 50  0000 C CNN
 F 2 "" H 4550 700 50  0001 C CNN
@@
 $EndComp
 $Comp
-L VSSA #PWR049
+L VSSA #PWR050
 U 1 1 5E15C764
 P 4550 2350
-F 0 "#PWR049" H 4550 2200 50  0001 C CNN
+F 0 "#PWR050" H 4550 2200 50  0001 C CNN
 F 1 "VSSA" V 4550 2550 50  0000 C CNN
 F 2 "" H 4550 2350 50  0001 C CNN
@@
 F 0 "C403" V 700 6300 50  0000 L CNN
 F 1 "47uF/16V/BP" V 800 6150 50  0000 L CNN
-F 2 "Capacitors_SMD:CP_Elec_5x5.7" H 950 6400 50  0001 C CNN
+F 2 "Capacitors_SMD:CP_Elec_8x5.4" H 950 6400 50  0001 C CNN
 F 3 "" H 950 6400 50  0001 C CNN
 	1    950  6400
@@
 	1850 1200 1700 1200
 $Comp
-L GNDA #PWR050
+L GNDA #PWR051
 U 1 1 5E2B3356
 P 1500 3800
-F 0 "#PWR050" H 1500 3550 50  0001 C CNN
+F 0 "#PWR051" H 1500 3550 50  0001 C CNN
 F 1 "GNDA" H 1500 3650 50  0000 C CNN
 F 2 "" H 1500 3800 50  0001 C CNN
@@
 $EndComp
 $Comp
-L GNDA #PWR051
+L GNDA #PWR052
 U 1 1 5E2B3754
 P 1200 7100
-F 0 "#PWR051" H 1200 6850 50  0001 C CNN
+F 0 "#PWR052" H 1200 6850 50  0001 C CNN
 F 1 "GNDA" H 1200 6950 50  0000 C CNN
 F 2 "" H 1200 7100 50  0001 C CNN
@@
 $EndComp
 $Comp
-L GNDA #PWR052
+L GNDA #PWR053
 U 1 1 5E2B38F6
 P 3050 6500
-F 0 "#PWR052" H 3050 6250 50  0001 C CNN
+F 0 "#PWR053" H 3050 6250 50  0001 C CNN
 F 1 "GNDA" H 3050 6350 50  0000 C CNN
 F 2 "" H 3050 6500 50  0001 C CNN
@@
 $EndComp
 $Comp
-L GNDA #PWR053
+L GNDA #PWR054
 U 1 1 5E2B3A31
 P 3300 6500
-F 0 "#PWR053" H 3300 6250 50  0001 C CNN
+F 0 "#PWR054" H 3300 6250 50  0001 C CNN
 F 1 "GNDA" H 3300 6350 50  0000 C CNN
 F 2 "" H 3300 6500 50  0001 C CNN
@@
 $EndComp
 $Comp
-L GNDA #PWR054
+L GNDA #PWR055
 U 1 1 5E2B3DBB
 P 9200 5700
-F 0 "#PWR054" H 9200 5450 50  0001 C CNN
+F 0 "#PWR055" H 9200 5450 50  0001 C CNN
 F 1 "GNDA" H 9200 5550 50  0000 C CNN
 F 2 "" H 9200 5700 50  0001 C CNN
@@
 $EndComp
 $Comp
-L GNDA #PWR055
+L GNDA #PWR056
 U 1 1 5E2B4029
 P 8300 5700
-F 0 "#PWR055" H 8300 5450 50  0001 C CNN
+F 0 "#PWR056" H 8300 5450 50  0001 C CNN
 F 1 "GNDA" H 8300 5550 50  0000 C CNN
 F 2 "" H 8300 5700 50  0001 C CNN
@@
 $EndComp
 $Comp
-L GNDA #PWR056
+L GNDA #PWR057
 U 1 1 5E2B47FD
 P 8300 3750
-F 0 "#PWR056" H 8300 3500 50  0001 C CNN
+F 0 "#PWR057" H 8300 3500 50  0001 C CNN
 F 1 "GNDA" H 8300 3600 50  0000 C CNN
 F 2 "" H 8300 3750 50  0001 C CNN
@@
 $EndComp
 $Comp
-L GNDA #PWR057
+L GNDA #PWR058
 U 1 1 5E2B4A01
 P 9200 3750
-F 0 "#PWR057" H 9200 3500 50  0001 C CNN
+F 0 "#PWR058" H 9200 3500 50  0001 C CNN
 F 1 "GNDA" H 9200 3600 50  0000 C CNN
 F 2 "" H 9200 3750 50  0001 C CNN
@@
 $EndComp
 $Comp
-L GNDA #PWR058
+L GNDA #PWR059
 U 1 1 5E2B50A9
 P 9200 1800
-F 0 "#PWR058" H 9200 1550 50  0001 C CNN
+F 0 "#PWR059" H 9200 1550 50  0001 C CNN
 F 1 "GNDA" H 9200 1650 50  0000 C CNN
 F 2 "" H 9200 1800 50  0001 C CNN
@@
 $EndComp
 $Comp
-L GNDA #PWR059
+L GNDA #PWR060
 U 1 1 5E2B5183
 P 8300 1800
-F 0 "#PWR059" H 8300 1550 50  0001 C CNN
+F 0 "#PWR060" H 8300 1550 50  0001 C CNN
 F 1 "GNDA" H 8300 1650 50  0000 C CNN
 F 2 "" H 8300 1800 50  0001 C CNN
@@
 $EndComp
 $Comp
-L GNDA #PWR060
+L GNDA #PWR061
 U 1 1 5E2B56AA
 P 5950 2000
-F 0 "#PWR060" H 5950 1750 50  0001 C CNN
+F 0 "#PWR061" H 5950 1750 50  0001 C CNN
 F 1 "GNDA" H 5950 1850 50  0000 C CNN
 F 2 "" H 5950 2000 50  0001 C CNN
@@
 $EndComp
 $Comp
-L GNDA #PWR061
+L GNDA #PWR062
 U 1 1 5E2B5784
 P 4700 1050
-F 0 "#PWR061" H 4700 800 50  0001 C CNN
+F 0 "#PWR062" H 4700 800 50  0001 C CNN
 F 1 "GNDA" H 4700 900 50  0000 C CNN
 F 2 "" H 4700 1050 50  0001 C CNN
@@
 $EndComp
 $Comp
-L GNDA #PWR062
+L GNDA #PWR063
 U 1 1 5E2B5A59
 P 4700 1950
-F 0 "#PWR062" H 4700 1700 50  0001 C CNN
+F 0 "#PWR063" H 4700 1700 50  0001 C CNN
 F 1 "GNDA" H 4700 1800 50  0000 C CNN
 F 2 "" H 4700 1950 50  0001 C CNN
@@
 $EndComp
 $Comp
-L GNDA #PWR063
+L GNDA #PWR064
 U 1 1 5E2B5D87
 P 2450 1200
-F 0 "#PWR063" H 2450 950 50  0001 C CNN
+F 0 "#PWR064" H 2450 950 50  0001 C CNN
 F 1 "GNDA" H 2450 1050 50  0000 C CNN
 F 2 "" H 2450 1200 50  0001 C CNN
@@
 $EndComp
 $Comp
-L GNDA #PWR064
+L GNDA #PWR065
 U 1 1 5E2B5E61
 P 2450 2000
-F 0 "#PWR064" H 2450 1750 50  0001 C CNN
+F 0 "#PWR065" H 2450 1750 50  0001 C CNN
 F 1 "GNDA" H 2450 1850 50  0000 C CNN
 F 2 "" H 2450 2000 50  0001 C CNN
@@
 $EndComp
 $Comp
-L GNDA #PWR065
+L GNDA #PWR066
 U 1 1 5E2B5F9F
 P 2450 2800
-F 0 "#PWR065" H 2450 2550 50  0001 C CNN
+F 0 "#PWR066" H 2450 2550 50  0001 C CNN
 F 1 "GNDA" H 2450 2650 50  0000 C CNN
 F 2 "" H 2450 2800 50  0001 C CNN
@@
 $EndComp
 $Comp
-L GNDA #PWR066
+L GNDA #PWR067
 U 1 1 5E2B61A3
 P 2450 3600
-F 0 "#PWR066" H 2450 3350 50  0001 C CNN
+F 0 "#PWR067" H 2450 3350 50  0001 C CNN
 F 1 "GNDA" H 2450 3450 50  0000 C CNN
 F 2 "" H 2450 3600 50  0001 C CNN
@@
 $EndComp
 $Comp
-L GNDA #PWR067
+L GNDA #PWR068
 U 1 1 5E2B6596
 P 5950 3950
-F 0 "#PWR067" H 5950 3700 50  0001 C CNN
+F 0 "#PWR068" H 5950 3700 50  0001 C CNN
 F 1 "GNDA" H 5950 3800 50  0000 C CNN
 F 2 "" H 5950 3950 50  0001 C CNN
@@
 $EndComp
 $Comp
-L GNDA #PWR068
+L GNDA #PWR069
 U 1 1 5E2B679A
 P 5950 5900
-F 0 "#PWR068" H 5950 5650 50  0001 C CNN
+F 0 "#PWR069" H 5950 5650 50  0001 C CNN
 F 1 "GNDA" H 5950 5750 50  0000 C CNN
 F 2 "" H 5950 5900 50  0001 C CNN
