File: bkm-129x.sch (KiCad schematic (older format))
At the start: 29 parts, among them IC010 LM2940CSX-5.0, IC050 LM2990SX-5.0, J001 Conn_02x32_Row_Letter_Last, Q501 DTC144EKA, U001 arduino-nano-v3, U502 74LVC125

Commit message: Minor adjustments
Parts:
- added MNT1, MNT2, MNT3, MNT4, MNT5: TEST_1P, Mounting_Holes:MountingHole_2.7mm_M2.5_DIN965_Pad, symbol TEST_1P
Connections:
- net GNDA: now also MNT1.1, MNT2.1, MNT3.1, MNT4.1, MNT5.1
Changed lines of the file:
@@
 Text Notes 1350 4400 2    60   ~ 0
 H_BLK
+$Comp
+L TEST_1P MNT1
+U 1 1 5E2D656F
+P 3750 6950
+F 0 "MNT1" H 3750 7220 50  0000 C CNN
+F 1 "TEST_1P" H 3750 7150 50  0000 C CNN
+F 2 "Mounting_Holes:MountingHole_2.7mm_M2.5_DIN965_Pad" H 3950 6950 50  0001 C CNN
+F 3 "" H 3950 6950 50  0001 C CNN
+	1    3750 6950
+	1    0    0    -1
+$EndComp
+$Comp
+L TEST_1P MNT2
+U 1 1 5E2D6718
+P 4100 6950
+F 0 "MNT2" H 4100 7220 50  0000 C CNN
+F 1 "TEST_1P" H 4100 7150 50  0000 C CNN
+F 2 "Mounting_Holes:MountingHole_2.7mm_M2.5_DIN965_Pad" H 4300 6950 50  0001 C CNN
+F 3 "" H 4300 6950 50  0001 C CNN
+	1    4100 6950
+	1    0    0    -1
+$EndComp
+$Comp
+L TEST_1P MNT3
+U 1 1 5E2D67A6
+P 4450 6950
+F 0 "MNT3" H 4450 7220 50  0000 C CNN
+F 1 "TEST_1P" H 4450 7150 50  0000 C CNN
+F 2 "Mounting_Holes:MountingHole_2.7mm_M2.5_DIN965_Pad" H 4650 6950 50  0001 C CNN
+F 3 "" H 4650 6950 50  0001 C CNN
+	1    4450 6950
+	1    0    0    -1
+$EndComp
+$Comp
+L TEST_1P MNT4
+U 1 1 5E2D6923
+P 4800 6950
+F 0 "MNT4" H 4800 7220 50  0000 C CNN
+F 1 "TEST_1P" H 4800 7150 50  0000 C CNN
+F 2 "Mounting_Holes:MountingHole_2.7mm_M2.5_DIN965_Pad" H 5000 6950 50  0001 C CNN
+F 3 "" H 5000 6950 50  0001 C CNN
+	1    4800 6950
+	1    0    0    -1
+$EndComp
+$Comp
+L GNDA #PWR044
+U 1 1 5E2D6BF3
+P 3750 6950
+F 0 "#PWR044" H 3750 6700 50  0001 C CNN
+F 1 "GNDA" V 3750 6750 50  0000 C CNN
+F 2 "" H 3750 6950 50  0001 C CNN
+F 3 "" H 3750 6950 50  0001 C CNN
+	1    3750 6950
+	1    0    0    -1
+$EndComp
+$Comp
+L GNDA #PWR045
+U 1 1 5E2D6C6A
+P 4100 6950
+F 0 "#PWR045" H 4100 6700 50  0001 C CNN
+F 1 "GNDA" V 4100 6750 50  0000 C CNN
+F 2 "" H 4100 6950 50  0001 C CNN
+F 3 "" H 4100 6950 50  0001 C CNN
+	1    4100 6950
+	1    0    0    -1
+$EndComp
+$Comp
+L GNDA #PWR046
+U 1 1 5E2D6CE1
+P 4450 6950
+F 0 "#PWR046" H 4450 6700 50  0001 C CNN
+F 1 "GNDA" V 4450 6750 50  0000 C CNN
+F 2 "" H 4450 6950 50  0001 C CNN
+F 3 "" H 4450 6950 50  0001 C CNN
+	1    4450 6950
+	1    0    0    -1
+$EndComp
+$Comp
+L GNDA #PWR047
+U 1 1 5E2D6DCE
+P 4800 6950
+F 0 "#PWR047" H 4800 6700 50  0001 C CNN
+F 1 "GNDA" V 4800 6750 50  0000 C CNN
+F 2 "" H 4800 6950 50  0001 C CNN
+F 3 "" H 4800 6950 50  0001 C CNN
+	1    4800 6950
+	1    0    0    -1
+$EndComp
+$Comp
+L TEST_1P MNT5
+U 1 1 5E2D7C05
+P 5150 6950
+F 0 "MNT5" H 5150 7220 50  0000 C CNN
+F 1 "TEST_1P" H 5150 7150 50  0000 C CNN
+F 2 "Mounting_Holes:MountingHole_2.7mm_M2.5_DIN965_Pad" H 5350 6950 50  0001 C CNN
+F 3 "" H 5350 6950 50  0001 C CNN
+	1    5150 6950
+	1    0    0    -1
+$EndComp
+$Comp
+L GNDA #PWR?
+U 1 1 5E2D7C0B
+P 5150 6950
+F 0 "#PWR?" H 5150 6700 50  0001 C CNN
+F 1 "GNDA" V 5150 6750 50  0000 C CNN
+F 2 "" H 5150 6950 50  0001 C CNN
+F 3 "" H 5150 6950 50  0001 C CNN
+	1    5150 6950
+	1    0    0    -1
+$EndComp
 $EndSCHEMATC

Commit message: Fixed some footprints
Parts:
- C501: footprint Capacitors_SMD:CP_Elec_6.3x4.5 -> Capacitors_SMD:CP_Elec_6.3x5.3
Changed lines of the file:
@@
 F 0 "C501" H 1710 5770 50  0000 L CNN
 F 1 "100uF" H 1710 5620 50  0000 L CNN
-F 2 "Capacitors_SMD:CP_Elec_6.3x4.5" H 1700 5700 50  0001 C CNN
+F 2 "Capacitors_SMD:CP_Elec_6.3x5.3" H 1700 5700 50  0001 C CNN
 F 3 "" H 1700 5700 50  0001 C CNN
 	1    1700 5700

Commit message: Added missing pullup resistor on SCLK
Parts:
- added R599: 4.7k, Resistors_SMD:R_0805_HandSoldering, symbol R_Small
Connections:
- net +5VD: now also R599.2
- net at U001.16 (17/PB5/PCINT5/SCK), U502.3 (O): now also R599.1
Changed lines of the file:
@@
 	1    0    0    -1
 $EndComp
+$Comp
+L R_Small R599
+U 1 1 5E4C37C4
+P 6000 3300
+F 0 "R599" H 6030 3320 50  0000 L CNN
+F 1 "4.7k" H 6030 3260 50  0000 L CNN
+F 2 "Resistors_SMD:R_0805_HandSoldering" H 6000 3300 50  0001 C CNN
+F 3 "" H 6000 3300 50  0001 C CNN
+	1    6000 3300
+	-1   0    0    1
+$EndComp
+$Comp
+L +5VD #PWR?
+U 1 1 5E4C3860
+P 6000 3150
+F 0 "#PWR?" H 6000 3000 50  0001 C CNN
+F 1 "+5VD" H 6000 3300 50  0000 C CNN
+F 2 "" H 6000 3150 50  0001 C CNN
+F 3 "" H 6000 3150 50  0001 C CNN
+	1    6000 3150
+	1    0    0    -1
+$EndComp
+Wire Wire Line
+	6000 3400 6000 3450
+Connection ~ 6000 3450
+Wire Wire Line
+	6000 3150 6000 3200
 $EndSCHEMATC
